Commit message: added mex cpp

File: urdf/rrbot.urdf (robot description, URDF)
Before this commit: robot rrbot, 4 links, 3 joints
Joints:
- joint ee_fixed_joint: origin xyz=1.0 0 0.0 rpy=0.0 0.0 0.0 -> xyz=1.0 0 0.1 rpy=0.0 0.0 0.0

Commit message: modified helpstr

File: urdf/rrbot.urdf (robot description, URDF)
Before this commit: robot rrbot, 4 links, 3 joints
Links:
- link ee_link: mass None -> 1e-6; geometry 
- link link1: geometry collision box size=1 0.1 0.1; visual box size=1 0.1 0.1
- link link2: geometry collision box size=1 0.1 0.1; visual box size=1 0.1 0.1
Joints:
- removed joint ee_fixed_joint
- added joint ee_joint: type fixed, parent link2, child ee_link, origin xyz=1 0 0.1 rpy=0 0 0, axis 0 0 1

Commit message: fixed bodyID error

File: urdf/rrbot.urdf (robot description, URDF)
Before this commit: robot rrbot, 4 links, 3 joints
Links:
- link link1: mass 1 -> 2
